Commit message: Add launch file to spawn my robot into the gazebo sim

File: src/simple_rover/urdf/simple_rover.urdf (robot description, URDF)
Before this commit: robot simple_rover, 6 links, 5 joints
Joints:
- joint front_left_wheel_joint: parent chassis -> base_link
- joint front_right_wheel_joint: parent chassis -> base_link
- joint rear_left_wheel_joint: parent chassis -> base_link
- joint rear_right_wheel_joint: parent chassis -> base_link
